Commit message: add drive_arc

File: mowbot_description/urdf/rl500.urdf.xacro (robot description, xacro)
@@ -134,5 +134,5 @@
   <xacro:macro name="wheel_size">
     <geometry>
-      <cylinder length="0.05" radius="0.127"/>
+      <cylinder length="0.005" radius="0.127"/>
     </geometry>
     <origin xyz="0 0 0" rpy="${M_PI/2} 0 0"/>

Commit message: publish joints, update URDF

File: mowbot_description/urdf/rl500.urdf.xacro (robot description, xacro)
@@ -187,8 +187,9 @@
   <joint name="imu_joint" type="fixed">
     <axis xyz="0 1 0" />
-    <origin xyz="0.279 0.05 0.342" rpy="0 0 0" />
+    <origin xyz="-0.18 0.08 0.07" rpy="0 0 0" />
     <parent link="base_link"/>
     <child link="imu"/>
   </joint>
+  <!-- No Lidar at present
   <link name="lidar">
     <xacro:sensor_visual/>
@@ -203,4 +204,5 @@
     <child link="lidar" />
   </joint>
+  -->
   <link name="gps">
     <xacro:sensor_visual/>
@@ -211,9 +213,11 @@
   </gazebo>
   <joint name="gps_joint" type="fixed">
-    <origin xyz="0.356 -0.102 0.342" rpy="0 0 0" />
+    <origin xyz="0.42 0.0 0.3" rpy="0 0 0" />
     <parent link="base_link" />
     <child link="gps" />
   </joint>
+  <!-- No Lidar at present -->
   <!-- hokuyo -->
+  <!--
   <gazebo reference="lidar">
     <sensor type="ray" name="head_hokuyo_sensor">
@@ -237,8 +241,10 @@
         <noise>
           <type>gaussian</type>
+  -->
           <!-- Noise parameters based on published spec for Hokuyo laser
                achieving "+-30mm" accuracy at range < 10m.  A mean of 0.0m and
                stddev of 0.01m will put 99.7% of samples within 0.03m of the true
                reading. -->
+  <!--
           <mean>0.0</mean>
           <stddev>0.01</stddev>
@@ -251,4 +257,5 @@
     </sensor>
     </gazebo>
+  -->
 	  <gazebo>
 	    <plugin name="imu_controller" filename="libgazebo_ros_imu.so">

Commit message: URDF updates

File: mowbot_description/urdf/rl500.urdf.xacro (robot description, xacro)
@@ -187,5 +187,5 @@
   <joint name="imu_joint" type="fixed">
     <axis xyz="0 1 0" />
-    <origin xyz="-0.18 0.08 0.07" rpy="0 0 0" />
+    <origin xyz="-0.18 -0.08 0.1" rpy="0 0 0" />
     <parent link="base_link"/>
     <child link="imu"/>
@@ -213,5 +213,5 @@
   </gazebo>
   <joint name="gps_joint" type="fixed">
-    <origin xyz="0.42 0.0 0.3" rpy="0 0 0" />
+    <origin xyz="0.42 0.0 0.35" rpy="0 0 0" />
     <parent link="base_link" />
     <child link="gps" />

Commit message: rename sensors to add _link

File: mowbot_description/urdf/rl500.urdf.xacro (robot description, xacro)
@@ -178,9 +178,9 @@
   <xacro:wheel prefix="left" reflect="1" />
   <xacro:wheel prefix="right" reflect="-1" />
-  <link name="imu">
+  <link name="imu_link">
     <xacro:sensor_visual/>
     <xacro:sensor_inertial/>
   </link>
-  <gazebo reference="imu">
+  <gazebo reference="imu_link">
     <material>Gazebo/Blue</material>
   </gazebo>
@@ -189,5 +189,5 @@
     <origin xyz="-0.18 -0.08 0.1" rpy="0 0 0" />
     <parent link="base_link"/>
-    <child link="imu"/>
+    <child link="imu_link"/>
   </joint>
   <!-- No Lidar at present
@@ -205,9 +205,9 @@
   </joint>
   -->
-  <link name="gps">
+  <link name="gps_link">
     <xacro:sensor_visual/>
     <xacro:sensor_inertial/>
   </link>
-  <gazebo reference="gps">
+  <gazebo reference="gps_link">
     <material>Gazebo/Blue</material>
   </gazebo>
@@ -215,5 +215,5 @@
     <origin xyz="0.42 0.0 0.35" rpy="0 0 0" />
     <parent link="base_link" />
-    <child link="gps" />
+    <child link="gps_link" />
   </joint>
   <!-- No Lidar at present -->
